Commit message: docs: 填写项目开发规范 + 修复雷达坐标系一致性描述
- backend spec: ESP32 下位机规范（目录结构、通讯协议、错误处理、日志、质量）
- frontend spec: ROS 上位机规范（目录结构、节点、Launch、参数/TF、URDF、质量）
- 更新 sensor_frame 描述：laser_frame 已在 URDF/驱动/costmap 中统一
- 添加 trellis 工作流配置和 claude 配置

Co-Authored-By: Claude Opus 4.6 (1M context) <noreply@anthropic.com>

File: Lin_ws/src/robot_description/urdf/robot_description.urdf (robot description, URDF)
Before this commit: robot robot_description, 6 links, 5 joints
Links:
- removed link laser_Link
- added link laser_frame, mass 0.094023; collision mesh filename=package://robot_description/meshes/laser_Link.STL; visual mesh filename=package://robot_description/meshes/laser_Link.STL
Joints:
- joint laser_joint: child laser_Link -> laser_frame
